File: kicad/PCIexpress_x1_half/PCIexpress_connector.kicad_sch (KiCad schematic)
At the start: 2 parts, among them J1 PCIexpress_bracket, J2 PCIexpress_x1

Commit message: update
Parts:
- J1: value PCIexpress_bracket -> (none); footprint PCIexpress:PCIexpress_bracket_full -> (none)
- J2: value PCIexpress_x1 -> (none); footprint PCIexpress:PCIexpress_x1 -> (none)
Other:
- title: PCIexpress_x1_full -> PCIexpress_x1_half
