File: kicad/PCIexpress_x1_half/PCIexpress_x1_half.kicad_sch (KiCad schematic)
At the start: 0 parts

Commit message: update
Other:
- title: PCIexpress_x1_full -> PCIexpress_x1_half
Changed lines of the file:
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@@
   (paper "A4")
   (title_block
-    (title "PCIexpress_x1_full")
+    (title "PCIexpress_x1_half")
     (company "Author: Luca Anastasio")
   )
-  (wire (pts (xy 31.75 36.83) (xy 34.29 36.83))
+  (wire (pts (xy 57.15 40.64) (xy 59.69 40.64))
+    (stroke (width 0) (type default) (color 0 0 0 0))
+  )
+  (wire (pts (xy 31.75 34.29) (xy 34.29 34.29))
     (stroke (width 0) (type default) (color 0 0 0 0))
   )
@@
     (stroke (width 0) (type default) (color 0 0 0 0))
   )
-  (wire (pts (xy 31.75 31.75) (xy 34.29 31.75))
-    (stroke (width 0) (type default) (color 0 0 0 0))
-  )
-  (wire (pts (xy 31.75 34.29) (xy 34.29 34.29))
-    (stroke (width 0) (type default) (color 0 0 0 0))
-  )
-  (wire (pts (xy 57.15 46.99) (xy 59.69 46.99))
-    (stroke (width 0) (type default) (color 0 0 0 0))
-  )
-  (wire (pts (xy 31.75 39.37) (xy 34.29 39.37))
+  (wire (pts (xy 31.75 58.42) (xy 34.29 58.42))
     (stroke (width 0) (type default) (color 0 0 0 0))
   )
@@
     (stroke (width 0) (type default) (color 0 0 0 0))
   )
-  (wire (pts (xy 31.75 60.96) (xy 34.29 60.96))
-    (stroke (width 0) (type default) (color 0 0 0 0))
-  )
-  (wire (pts (xy 31.75 29.21) (xy 34.29 29.21))
-    (stroke (width 0) (type default) (color 0 0 0 0))
-  )
   (wire (pts (xy 57.15 35.56) (xy 59.69 35.56))
-    (stroke (width 0) (type default) (color 0 0 0 0))
-  )
-  (wire (pts (xy 57.15 40.64) (xy 59.69 40.64))
-    (stroke (width 0) (type default) (color 0 0 0 0))
-  )
-  (wire (pts (xy 31.75 46.99) (xy 34.29 46.99))
     (stroke (width 0) (type default) (color 0 0 0 0))
   )
@@
     (stroke (width 0) (type default) (color 0 0 0 0))
   )
+  (wire (pts (xy 57.15 58.42) (xy 59.69 58.42))
+    (stroke (width 0) (type default) (color 0 0 0 0))
+  )
+  (wire (pts (xy 31.75 29.21) (xy 34.29 29.21))
+    (stroke (width 0) (type default) (color 0 0 0 0))
+  )
   (wire (pts (xy 57.15 60.96) (xy 59.69 60.96))
+    (stroke (width 0) (type default) (color 0 0 0 0))
+  )
+  (wire (pts (xy 31.75 43.18) (xy 34.29 43.18))
+    (stroke (width 0) (type default) (color 0 0 0 0))
+  )
+  (wire (pts (xy 31.75 39.37) (xy 34.29 39.37))
+    (stroke (width 0) (type default) (color 0 0 0 0))
+  )
+  (wire (pts (xy 31.75 46.99) (xy 34.29 46.99))
+    (stroke (width 0) (type default) (color 0 0 0 0))
+  )
+  (wire (pts (xy 31.75 31.75) (xy 34.29 31.75))
+    (stroke (width 0) (type default) (color 0 0 0 0))
+  )
+  (wire (pts (xy 31.75 36.83) (xy 34.29 36.83))
+    (stroke (width 0) (type default) (color 0 0 0 0))
+  )
+  (wire (pts (xy 57.15 53.34) (xy 59.69 53.34))
+    (stroke (width 0) (type default) (color 0 0 0 0))
+  )
+  (wire (pts (xy 31.75 60.96) (xy 34.29 60.96))
     (stroke (width 0) (type default) (color 0 0 0 0))
   )
@@
     (stroke (width 0) (type default) (color 0 0 0 0))
   )
-  (wire (pts (xy 57.15 58.42) (xy 59.69 58.42))
+  (wire (pts (xy 57.15 46.99) (xy 59.69 46.99))
     (stroke (width 0) (type default) (color 0 0 0 0))
   )
-  (wire (pts (xy 57.15 53.34) (xy 59.69 53.34))
-    (stroke (width 0) (type default) (color 0 0 0 0))
-  )
-  (wire (pts (xy 31.75 58.42) (xy 34.29 58.42))
-    (stroke (width 0) (type default) (color 0 0 0 0))
-  )
-  (wire (pts (xy 31.75 43.18) (xy 34.29 43.18))
-    (stroke (width 0) (type default) (color 0 0 0 0))
-  )
-  (label "~{PRSNT2x8}" (at 31.75 36.83 180)
+  (label "~{WAKE}" (at 31.75 46.99 180)
     (effects (font (size 1.27 1.27)) (justify right bottom))
   )
-  (label "~{TRST}" (at 59.69 43.18 0)
+  (label "REFCLK+" (at 59.69 50.8 0)
+    (effects (font (size 1.27 1.27)) (justify left bottom))
+  )
+  (label "TMS" (at 59.69 35.56 0)
+    (effects (font (size 1.27 1.27)) (justify left bottom))
+  )
+  (label "PER0_P" (at 31.75 58.42 180)
+    (effects (font (size 1.27 1.27)) (justify right bottom))
+  )
+  (label "~{PERST}" (at 59.69 46.99 0)
+    (effects (font (size 1.27 1.27)) (justify left bottom))
+  )
+  (label "SMDAT" (at 31.75 53.34 180)
+    (effects (font (size 1.27 1.27)) (justify right bottom))
+  )
+  (label "TDO" (at 31.75 43.18 180)
+    (effects (font (size 1.27 1.27)) (justify right bottom))
+  )
+  (label "REFCLK-" (at 59.69 53.34 0)
     (effects (font (size 1.27 1.27)) (justify left bottom))
   )
@@
     (effects (font (size 1.27 1.27)) (justify left bottom))
   )
-  (label "~{PRSNT2x4}" (at 31.75 34.29 180)
+  (label "~{PRSNT2x1}" (at 31.75 31.75 180)
     (effects (font (size 1.27 1.27)) (justify right bottom))
+  )
+  (label "TCK" (at 59.69 38.1 0)
+    (effects (font (size 1.27 1.27)) (justify left bottom))
   )
   (label "~{PRSNT2x16}" (at 31.75 39.37 180)
     (effects (font (size 1.27 1.27)) (justify right bottom))
   )
-  (label "REFCLK+" (at 59.69 50.8 0)
-    (effects (font (size 1.27 1.27)) (justify left bottom))
-  )
   (label "SMCLK" (at 31.75 50.8 180)
-    (effects (font (size 1.27 1.27)) (justify right bottom))
-  )
-  (label "PER0_P" (at 31.75 58.42 180)
-    (effects (font (size 1.27 1.27)) (justify right bottom))
-  )
-  (label "REFCLK-" (at 59.69 53.34 0)
-    (effects (font (size 1.27 1.27)) (justify left bottom))
-  )
-  (label "TCK" (at 59.69 38.1 0)
-    (effects (font (size 1.27 1.27)) (justify left bottom))
-  )
-  (label "~{WAKE}" (at 31.75 46.99 180)
-    (effects (font (size 1.27 1.27)) (justify right bottom))
-  )
-  (label "TDO" (at 31.75 43.18 180)
-    (effects (font (size 1.27 1.27)) (justify right bottom))
-  )
-  (label "SMDAT" (at 31.75 53.34 180)
-    (effects (font (size 1.27 1.27)) (justify right bottom))
-  )
-  (label "~{PRSNT2x1}" (at 31.75 31.75 180)
     (effects (font (size 1.27 1.27)) (justify right bottom))
   )
@@
     (effects (font (size 1.27 1.27)) (justify left bottom))
   )
-  (label "~{PRSNT1}" (at 31.75 29.21 180)
-    (effects (font (size 1.27 1.27)) (justify right bottom))
-  )
-  (label "TMS" (at 59.69 35.56 0)
+  (label "~{TRST}" (at 59.69 43.18 0)
     (effects (font (size 1.27 1.27)) (justify left bottom))
   )
-  (label "~{PERST}" (at 59.69 46.99 0)
-    (effects (font (size 1.27 1.27)) (justify left bottom))
+  (label "PER0_N" (at 31.75 60.96 180)
+    (effects (font (size 1.27 1.27)) (justify right bottom))
   )
   (label "PET0_N" (at 59.69 60.96 0)
     (effects (font (size 1.27 1.27)) (justify left bottom))
   )
-  (label "PER0_N" (at 31.75 60.96 180)
+  (label "~{PRSNT1}" (at 31.75 29.21 180)
+    (effects (font (size 1.27 1.27)) (justify right bottom))
+  )
+  (label "~{PRSNT2x8}" (at 31.75 36.83 180)
+    (effects (font (size 1.27 1.27)) (justify right bottom))
+  )
+  (label "~{PRSNT2x4}" (at 31.75 34.29 180)
     (effects (font (size 1.27 1.27)) (justify right bottom))
   )
@@
       (effects (font (size 1.27 1.27)) (justify left bottom))
     )
-    (property "Sheet file" "PCIexpress_connector.kicad_sch" (id 1) (at 27.94 64.77 0)
+    (property "Sheet file" "PCIexpress_connector.kicad_sch" (id 1) (at 31.75 64.77 0)
       (effects (font (size 1.27 1.27)) (justify left top))
     )
