File: kicad/PCIexpress_x1_half/term.kicad_sch (KiCad schematic)
At the start: 2 parts

Commit message: update
Parts:
- R1, R2: value 49.9 -> (none); footprint Resistor_SMD:R_0603_1608Metric -> (none)
Other:
- title: PCIexpress_x1_full -> PCIexpress_x1_half
Changed lines of the file:
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@@
   (paper "A4")
   (title_block
-    (title "PCIexpress_x1_full")
+    (title "PCIexpress_x1_half")
     (company "Author: Luca Anastasio")
+  )
+  (junction (at 146.05 90.17) (diameter 0) (color 0 0 0 0)
   )
   (junction (at 120.65 90.17) (diameter 0) (color 0 0 0 0)
   )
-  (junction (at 146.05 90.17) (diameter 0) (color 0 0 0 0)
+  (wire (pts (xy 118.11 90.17) (xy 120.65 90.17))
+    (stroke (width 0) (type default) (color 0 0 0 0))
   )
-  (wire (pts (xy 146.05 92.71) (xy 146.05 90.17))
+  (wire (pts (xy 146.05 100.33) (xy 146.05 102.87))
+    (stroke (width 0) (type default) (color 0 0 0 0))
+  )
+  (wire (pts (xy 120.65 90.17) (xy 123.19 90.17))
+    (stroke (width 0) (type default) (color 0 0 0 0))
+  )
+  (wire (pts (xy 120.65 100.33) (xy 120.65 102.87))
+    (stroke (width 0) (type default) (color 0 0 0 0))
+  )
+  (wire (pts (xy 120.65 92.71) (xy 120.65 90.17))
     (stroke (width 0) (type default) (color 0 0 0 0))
   )
@@
     (stroke (width 0) (type default) (color 0 0 0 0))
   )
-  (wire (pts (xy 120.65 100.33) (xy 120.65 102.87))
-    (stroke (width 0) (type default) (color 0 0 0 0))
-  )
   (wire (pts (xy 146.05 90.17) (xy 148.59 90.17))
     (stroke (width 0) (type default) (color 0 0 0 0))
   )
-  (wire (pts (xy 120.65 92.71) (xy 120.65 90.17))
+  (wire (pts (xy 146.05 92.71) (xy 146.05 90.17))
     (stroke (width 0) (type default) (color 0 0 0 0))
-  )
-  (wire (pts (xy 118.11 90.17) (xy 120.65 90.17))
-    (stroke (width 0) (type default) (color 0 0 0 0))
-  )
-  (wire (pts (xy 120.65 90.17) (xy 123.19 90.17))
-    (stroke (width 0) (type default) (color 0 0 0 0))
-  )
-  (wire (pts (xy 146.05 100.33) (xy 146.05 102.87))
-    (stroke (width 0) (type default) (color 0 0 0 0))
-  )
-  (hierarchical_label "OUT-" (shape output) (at 118.11 90.17 180)
-    (effects (font (size 1.27 1.27)) (justify right))
   )
   (hierarchical_label "IN+" (shape input) (at 148.59 90.17 0)
@@
   (hierarchical_label "IN-" (shape input) (at 123.19 90.17 0)
     (effects (font (size 1.27 1.27)) (justify left))
+  )
+  (hierarchical_label "OUT-" (shape output) (at 118.11 90.17 180)
+    (effects (font (size 1.27 1.27)) (justify right))
   )
   (hierarchical_label "OUT+" (shape output) (at 143.51 90.17 180)
@@
       (effects (font (size 1.27 1.27)) (justify left))
     )
-    (property "Value" "49.9" (id 1) (at 122.428 97.663 0)
+    (property "Value" "" (id 1) (at 122.428 97.663 0)
       (effects (font (size 1.27 1.27)) (justify left))
     )
-    (property "Footprint" "Resistor_SMD:R_0603_1608Metric" (id 2) (at 118.872 96.52 90)
+    (property "Footprint" "" (id 2) (at 118.872 96.52 90)
       (effects (font (size 1.27 1.27)) hide)
     )
@@
       (effects (font (size 1.27 1.27)) (justify left))
     )
-    (property "Value" "49.9" (id 1) (at 147.828 97.663 0)
+    (property "Value" "" (id 1) (at 147.828 97.663 0)
       (effects (font (size 1.27 1.27)) (justify left))
     )
-    (property "Footprint" "Resistor_SMD:R_0603_1608Metric" (id 2) (at 144.272 96.52 90)
+    (property "Footprint" "" (id 2) (at 144.272 96.52 90)
       (effects (font (size 1.27 1.27)) hide)
     )
@@
       (effects (font (size 1.27 1.27)) hide)
     )
-    (property "Value" "GND" (id 1) (at 120.777 107.2642 0))
+    (property "Value" "" (id 1) (at 120.777 107.2642 0))
     (property "Footprint" "" (id 2) (at 120.65 102.87 0)
       (effects (font (size 1.27 1.27)) hide)
@@
       (effects (font (size 1.27 1.27)) hide)
     )
-    (property "Value" "GND" (id 1) (at 146.177 107.2642 0))
+    (property "Value" "" (id 1) (at 146.177 107.2642 0))
     (property "Footprint" "" (id 2) (at 146.05 102.87 0)
       (effects (font (size 1.27 1.27)) hide)
