File: kicad/PCIexpress_x16_low/decap.kicad_sch (KiCad schematic)
At the start: 2 parts

Commit message: fix
Parts:
- C? (x2): value (none) -> ~
Changed lines of the file:
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@@
     (in_bom yes) (on_board yes)
     (property "Reference" "C?" (id 0) (at 160.02 74.8792 90))
-    (property "Value" "" (id 1) (at 160.02 77.1906 90))
+    (property "Value" "~" (id 1) (at 160.02 77.1906 90))
     (property "Footprint" "" (id 2) (at 156.21 82.2452 0)
       (effects (font (size 1.27 1.27)) hide)
@@
     (in_bom yes) (on_board yes)
     (property "Reference" "C?" (id 0) (at 160.02 87.5792 90))
-    (property "Value" "" (id 1) (at 160.02 89.8906 90))
+    (property "Value" "~" (id 1) (at 160.02 89.8906 90))
     (property "Footprint" "" (id 2) (at 163.83 94.9452 0)
       (effects (font (size 1.27 1.27)) hide)
