File: kicad/PCIexpress_x16_low/term.kicad_sch (KiCad schematic)
At the start: 2 parts

Commit message: fix
Parts:
- R1, R2: value (none) -> ~
Changed lines of the file:
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@@
       (effects (font (size 1.27 1.27)) (justify left))
     )
-    (property "Value" "" (id 1) (at 122.428 97.663 0)
+    (property "Value" "~" (id 1) (at 122.428 97.663 0)
       (effects (font (size 1.27 1.27)) (justify left))
     )
@@
       (effects (font (size 1.27 1.27)) (justify left))
     )
-    (property "Value" "" (id 1) (at 147.828 97.663 0)
+    (property "Value" "~" (id 1) (at 147.828 97.663 0)
       (effects (font (size 1.27 1.27)) (justify left))
     )
@@
       (effects (font (size 1.27 1.27)) hide)
     )
-    (property "Value" "" (id 1) (at 120.777 107.2642 0))
+    (property "Value" "~" (id 1) (at 120.777 107.2642 0))
     (property "Footprint" "" (id 2) (at 120.65 102.87 0)
       (effects (font (size 1.27 1.27)) hide)
@@
       (effects (font (size 1.27 1.27)) hide)
     )
-    (property "Value" "" (id 1) (at 146.177 107.2642 0))
+    (property "Value" "~" (id 1) (at 146.177 107.2642 0))
     (property "Footprint" "" (id 2) (at 146.05 102.87 0)
       (effects (font (size 1.27 1.27)) hide)
