File: kicad/PCIexpress_x1_full/PCIexpress_connector.kicad_sch (KiCad schematic)
At the start: 2 parts, among them J1 PCIexpress_bracket, J2 PCIexpress_x1

Commit message: update
Changed lines of the file:
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@@
   )
   (text "From add-in card transmitter to mainboard receiver\nPlace AC coupling capacitors here if necessary"
-    (at 139.7 55.88 0)
+    (at 143.51 17.78 0)
     (effects (font (size 1.27 1.27)) (justify left bottom))
   )
   (text "From mainboard transmitter to add-in card receiver\nPlace termination resistors here if necessary"
-    (at 66.04 20.32 0)
+    (at 64.77 16.51 0)
     (effects (font (size 1.27 1.27)) (justify right bottom))
   )
